Commit message: ps4 controller and urdf fixed

File: src/smoothop/urdf/smoothop.urdf (robot description, URDF)
Before this commit: robot smoothoperator, 3 links, 3 joints
Links:
- link base_link: geometry visual box size=0.3 0.2 0.1
- link laser: geometry visual cylinder length=0.04 radius=0.035
Joints:
- removed joint base_link
- joint laser_joint: origin xyz=0 0 0.2 rpy=0 0 -1.57 -> xyz=0.15 0 0.1 rpy=0 0 0
